File: rev_a/hail.sch (EAGLE design)
At the start: 72 parts, among them J1 MICRO_USB_B_HIROSE_ZX62R-B-5P, J2 TC2030-JLINK-NL_NOSILK, J3 TC2030-JLINK-NL_NOSILK, U1 FT231XQ, U2 FXOS8700CQ, U3 ISL29035, U4 MAX8887EZK33+T, U5 NRF51822QF, U6 SAM4LC8BA, U7 SI7021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

Commit message: Update mistaken digikey part numbers
Parts:
- U5: DIGIKEY (none) -> 1490-1049-1-ND
- U6: DIGIKEY (none) -> ATSAM4LC8BA-MURCT-ND
- U7: DIGIKEY (none) -> 336-3141-ND
Changed lines of the file:
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@@
 <attribute name="TITLE" value="Hail"/>
 </part>
-<part name="U5" library="chips" deviceset="NRF51822" device="QF"/>
+<part name="U5" library="chips" deviceset="NRF51822" device="QF">
+<attribute name="DIGIKEY" value="1490-1049-1-ND"/>
+<attribute name="MOUSER" value=""/>
+</part>
 <part name="J1" library="connector" deviceset="MICRO_USB_B_HIROSE_ZX62R-B-5P" device="">
 <attribute name="DIGIKEY" value="H125274CT-ND"/>
@@
 <attribute name="TITLE" value="Hail"/>
 </part>
-<part name="U7" library="chips" deviceset="SI7021" device=""/>
+<part name="U7" library="chips" deviceset="SI7021" device="">
+<attribute name="DIGIKEY" value="336-3141-ND"/>
+</part>
 <part name="R6" library="passives" deviceset="RESISTOR" device="0402_RES" value="10k">
 <attribute name="DIGIKEY" value="1276-3431-1-ND"/>
@@
 <part name="P+14" library="supply1" deviceset="VCC" device=""/>
 <part name="GND23" library="umich" deviceset="GND" device=""/>
-<part name="U6" library="chips" deviceset="SAM4LC8BA" device=""/>
+<part name="U6" library="chips" deviceset="SAM4LC8BA" device="">
+<attribute name="DIGIKEY" value="ATSAM4LC8BA-MURCT-ND"/>
+</part>
 <part name="GND27" library="umich" deviceset="GND" device=""/>
 <part name="C18" library="passives" deviceset="CAPACITOR" device="0402_CAP" value="100nF">
