File: hardware/hail/rev_a/hail.brd (EAGLE design)
At the start: 20.3 x 36.6 mm, 75 parts, among them J1 MICRO_USB_B_HIROSE_ZX62R-B-5P, J2 TC2030-JLINK-NL_NOSILK, J3 TC2030-JLINK-NL_NOSILK, U1 FT231XQ, U2 FXOS8700CQ, U3 ISL29035, U4 MAX8887EZK33+T, U5 NRF51822QF, U6 SAM4LC8BA, U7 SI7021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

Commit message: Fix mistaken pin names and BOM parts
Pins:

 * fix RGB led pins
 * correct mapping of NRF_RTS/CTS pins

BOM:

 * FB1 was 0603 by mistake. Picked 0402 package
 * Found part for 12-pin headers for Hail
Connections:
- net BLUE_LED: now also R2.1, U6.41; no longer R1.1, U6.40
- net GREEN_LED: now also R3.1, U6.42; no longer R2.1, U6.41
- net NRF_CTS: now also TP1.TP, U5.17, U6.27; no longer TP2.TP, U5.18, U6.28
- net NRF_RTS: now also TP2.TP, U5.18, U6.28; no longer TP1.TP, U5.17, U6.27
- net RED_LED: now also R1.1, U6.40; no longer R3.1, U6.42
Routing:
- net NRF_RTS: track 23.5 -> 18.2 mm
- net NRF_CTS: track 18.2 -> 23.5 mm
- net RED_LED: track 10.7 -> 11.5 mm
- net GREEN_LED: track 11.2 -> 10.7 mm
Changed lines of the file:
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@@
 <attribute name="NAME" x="9.9568" y="5.5238" size="0.508" layer="25" font="vector" ratio="18" rot="R180" align="bottom-center"/>
 </element>
-<element name="JP3" library="Particle" package="1X12-CASTELLATED" value="M12PTH-CST-L" x="1.27" y="18.288" smashed="yes" rot="R180"/>
-<element name="JP4" library="Particle" package="1X12-CASTELLATED" value="M12PTH-CST-R" x="19.05" y="18.288" smashed="yes"/>
+<element name="JP3" library="Particle" package="1X12-CASTELLATED" value="M12PTH-CST-L" x="1.27" y="18.288" smashed="yes" rot="R180">
+<attribute name="DIGIKEY" value="S1011E-12-ND" x="1.27" y="18.288" size="1.778" layer="27" rot="R180" display="off"/>
+</element>
+<element name="JP4" library="Particle" package="1X12-CASTELLATED" value="M12PTH-CST-R" x="19.05" y="18.288" smashed="yes">
+<attribute name="DIGIKEY" value="S1011E-12-ND" x="19.05" y="18.288" size="1.778" layer="27" display="off"/>
+</element>
 <element name="U1" library="chips" package="QFN-20-4MM" value="FT231XQ" x="10.16" y="28.956" smashed="yes" rot="R180">
 <attribute name="MPN" value="FT231XQ-R" x="10.16" y="28.956" size="1.778" layer="27" rot="R180" display="off"/>
@@
 </element>
 <element name="FB1" library="passives" package="0402_CAP" value="1.5k" x="3.81" y="18.288" smashed="yes" rot="R270">
-<attribute name="DIGIKEY" value="490-5216-1-ND" x="1.016" y="17.272" size="1.778" layer="27" rot="R270" display="off"/>
+<attribute name="DIGIKEY" value="1276-6395-1-ND" x="1.016" y="17.272" size="1.778" layer="27" rot="R270" display="off"/>
 <attribute name="NAME" x="3.7084" y="19.8628" size="0.508" layer="25" font="vector" ratio="18" rot="R270" align="bottom-center"/>
 </element>
@@
 <wire x1="10.16" y1="32.451" x2="10.16" y2="30.856" width="0.2032" layer="1"/>
 </signal>
-<signal name="BLUE_LED">
+<signal name="RED_LED">
 <contactref element="R1" pad="1"/>
 <contactref element="U6" pad="40"/>
@@
 <wire x1="15.94993125" y1="11.25093125" x2="15.94993125" y2="11.43" width="0.2032" layer="1"/>
 </signal>
-<signal name="GREEN_LED">
+<signal name="BLUE_LED">
 <contactref element="R2" pad="1"/>
 <contactref element="U6" pad="41"/>
@@
 <wire x1="14.732" y1="10.7696" x2="15.1892" y2="11.2268" width="0.2032" layer="16"/>
 </signal>
-<signal name="RED_LED">
+<signal name="GREEN_LED">
 <contactref element="R3" pad="1"/>
 <contactref element="U6" pad="42"/>
@@
 <wire x1="9.0678" y1="27.8638" x2="8.4582" y2="28.2702" width="0.2032" layer="16"/>
 </signal>
-<signal name="NRF_RTS">
+<signal name="NRF_CTS">
 <contactref element="U6" pad="27"/>
 <contactref element="U5" pad="17"/>
@@
 <wire x1="5.9182" y1="20.828" x2="6.5532" y2="21.463" width="0.2032" layer="16"/>
 </signal>
-<signal name="NRF_CTS">
+<signal name="NRF_RTS">
 <contactref element="U6" pad="28"/>
 <contactref element="U5" pad="18"/>
