File: hardware/hail/rev_a/hail.sch (EAGLE design)
At the start: 72 parts, among them J1 MICRO_USB_B_HIROSE_ZX62R-B-5P, J2 TC2030-JLINK-NL_NOSILK, J3 TC2030-JLINK-NL_NOSILK, U1 FT231XQ, U2 FXOS8700CQ, U3 ISL29035, U4 MAX8887EZK33+T, U5 NRF51822QF, U6 SAM4LC8BA, U7 SI7021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

Commit message: Fix mistaken pin names and BOM parts
Pins:

 * fix RGB led pins
 * correct mapping of NRF_RTS/CTS pins

BOM:

 * FB1 was 0603 by mistake. Picked 0402 package
 * Found part for 12-pin headers for Hail
Parts:
- FB1: DIGIKEY 490-5216-1-ND -> 1276-6395-1-ND
- JP3, JP4: DIGIKEY (none) -> S1011E-12-ND
Connections:
- net BLUE_LED: now also R2.1, U6.PA14; no longer R1.1, U6.PA13
- net GREEN_LED: now also R3.1, U6.PA15; no longer R2.1, U6.PA14
- net NRF_CTS: now also TP1.TP, U5.P11, U6.PB06; no longer TP2.TP, U5.P12, U6.PB07
- net NRF_RTS: now also TP2.TP, U5.P12, U6.PB07; no longer TP1.TP, U5.P11, U6.PB06
- net RED_LED: now also R1.1, U6.PA13; no longer R3.1, U6.PA15
Changed lines of the file:
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@@
 <part name="A1" library="chips" deviceset="FRACTUS-2.4GHZ-FR05-S1-N-0-110" device=""/>
 <part name="B1" library="chips" deviceset="BAL-NRF01D3" device=""/>
-<part name="JP3" library="Particle" deviceset="M12" device="PTH-CST-L"/>
-<part name="JP4" library="Particle" deviceset="M12" device="PTH-CST-R"/>
+<part name="JP3" library="Particle" deviceset="M12" device="PTH-CST-L">
+<attribute name="DIGIKEY" value="S1011E-12-ND"/>
+</part>
+<part name="JP4" library="Particle" deviceset="M12" device="PTH-CST-R">
+<attribute name="DIGIKEY" value="S1011E-12-ND"/>
+</part>
 <part name="U1" library="chips" deviceset="FT231X" device="Q"/>
 <part name="GND1" library="supply1" deviceset="GND" device=""/>
@@
 </part>
 <part name="FB1" library="passives" deviceset="FERRITE_BEAD" device="0402" value="1.5k">
-<attribute name="DIGIKEY" value="490-5216-1-ND"/>
+<attribute name="DIGIKEY" value="1276-6395-1-ND"/>
 </part>
 <part name="C22" library="passives" deviceset="CAPACITOR" device="0402_CAP" value="100nF">
@@
 </instance>
 <instance part="P+1" gate="VCC" x="187.96" y="162.56"/>
-<instance part="JP3" gate="G$1" x="226.06" y="91.44" rot="MR0"/>
-<instance part="JP4" gate="G$1" x="226.06" y="50.8" rot="MR0"/>
+<instance part="JP3" gate="G$1" x="226.06" y="91.44" rot="MR0">
+<attribute name="DIGIKEY" x="226.06" y="91.44" size="1.778" layer="96" rot="MR0" display="off"/>
+</instance>
+<instance part="JP4" gate="G$1" x="226.06" y="50.8" rot="MR0">
+<attribute name="DIGIKEY" x="226.06" y="50.8" size="1.778" layer="96" rot="MR0" display="off"/>
+</instance>
 <instance part="S1" gate="G$1" x="111.76" y="58.42"/>
 <instance part="S2" gate="G$1" x="111.76" y="27.94"/>
@@
 </segment>
 </net>
-<net name="BLUE_LED" class="0">
+<net name="RED_LED" class="0">
 <segment>
 <pinref part="R1" gate="G$1" pin="1"/>
@@
 </segment>
 </net>
-<net name="GREEN_LED" class="0">
+<net name="BLUE_LED" class="0">
 <segment>
 <pinref part="R2" gate="G$1" pin="1"/>
@@
 </segment>
 </net>
-<net name="RED_LED" class="0">
+<net name="GREEN_LED" class="0">
 <segment>
 <pinref part="R3" gate="G$1" pin="1"/>
@@
 </segment>
 </net>
-<net name="NRF_RTS" class="0">
+<net name="NRF_CTS" class="0">
 <segment>
 <pinref part="U6" gate="G$1" pin="PB06"/>
@@
 </segment>
 </net>
-<net name="NRF_CTS" class="0">
+<net name="NRF_RTS" class="0">
 <segment>
 <pinref part="U6" gate="G$1" pin="PB07"/>
@@
 </segment>
 </net>
-<net name="NRF_RTS" class="0">
+<net name="NRF_CTS" class="0">
 <segment>
 <label x="78.74" y="93.98" size="1.27" layer="95" font="vector" rot="R180" xref="yes"/>
@@
 </segment>
 </net>
-<net name="NRF_CTS" class="0">
+<net name="NRF_RTS" class="0">
 <segment>
 <label x="78.74" y="91.44" size="1.27" layer="95" font="vector" rot="R180" xref="yes"/>
