File: hardware/hail-debug/rev_a/hail-debug.brd (EAGLE design)
At the start: 61 x 63.5 mm, 58 parts, among them J1 MILLMAX_0985-X-15-20-71-14-11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, J10 MILLMAX_0985-X-15-20-71-14-11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, J11 MILLMAX_0985-X-15-20-71-14-11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, J12 MILLMAX_0985-X-15-20-71-14-11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, J13 MILLMAX_0985-X-15-20-71-14-11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, J14 MILLMAX_0908-X-15-20-75-14-11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, J15 MILLMAX_0908-X-15-20-75-14-11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, J16 MILLMAX_0908-X-15-20-75-14-11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, J17 MILLMAX_0908-X-15-20-75-14-11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, J18 MILLMAX_0908-X-15-20-75-14-11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, J19 MILLMAX_0908-X-15-20-75-14-11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, J2 MILLMAX_0985-X-15-20-71-14-11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, J20 MILLMAX_0908-X-15-20-75-14-11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, J21 MILLMAX_0908-X-15-20-75-14-11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, J22 MILLMAX_0908-X-15-20-75-14-11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, J23 MILLMAX_0908-X-15-20-75-14-11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, J24 MILLMAX_0908-X-15-20-75-14-11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, J25 MILLMAX_0908-X-15-20-75-14-11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, J26 MILLMAX_0908-X-15-20-75-14-11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, J27 MILLMAX_0908-X-15-20-75-14-11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, J28 MILLMAX_0908-X-15-20-75-14-11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, J29 MILLMAX_0908-X-15-20-75-14-11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, J3 MILLMAX_0985-X-15-20-71-14-11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, J30 MILLMAX_0908-X-15-20-75-14-11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, J31 MILLMAX_0908-X-15-20-75-14-11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, J32 MILLMAX_0908-X-15-20-75-14-11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, J33 MILLMAX_0908-X-15-20-75-14-11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, J34 MILLMAX_0908-X-15-20-75-14-11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, J35 MILLMAX_0908-X-15-20-75-14-11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, J36 MILLMAX_0908-X-15-20-75-14-11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, J37 MILLMAX_0908-X-15-20-75-14-11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, J38 MILLMAX_0985-X-15-20-71-14-11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, J39 MILLMAX_0985-X-15-20-71-14-11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, J4 MILLMAX_0985-X-15-20-71-14-11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, J40 MILLMAX_0985-X-15-20-71-14-11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, J41 MILLMAX_0985-X-15-20-71-14-11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, J42 MILLMAX_0985-X-15-20-71-14-11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, J43 MILLMAX_0985-X-15-20-71-14-11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, J44 TC2030-JLINK-L, J46 SCREW_TERMINAL_12_0.100, J47 SCREW_TERMINAL_12_0.100, J5 MILLMAX_0985-X-15-20-71-14-11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, J50 SCREW-TERMINAL_7_0.100, J51 SCREW-TERMINAL_7_0.100, J6 MILLMAX_0985-X-15-20-71-14-11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, J7 MILLMAX_0985-X-15-20-71-14-11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, J8 MILLMAX_0985-X-15-20-71-14-11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, J9 MILLMAX_0985-X-15-20-71-14-11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

Commit message: small fixes
Parts:
- renumbered JP1 to J52
Changed lines of the file:
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@@
 <element name="H3" library="holes" package="3,2" value="MOUNT-HOLE3.2" x="36.83" y="-17.78"/>
 <element name="H4" library="holes" package="3,2" value="MOUNT-HOLE3.2" x="-16.51" y="-17.78"/>
-<element name="JP1" library="pinhead" package="2X14" value="" x="10.16" y="-11.43" smashed="yes">
+<element name="J52" library="pinhead" package="2X14" value="" x="10.16" y="-11.43" smashed="yes">
 <attribute name="VALUE" x="-7.62" y="-15.875" size="1.27" layer="27"/>
 </element>
@@
 <signal name="!LIGHT_INT">
 <contactref element="J13" pad="P1"/>
-<contactref element="JP1" pad="27"/>
-<contactref element="JP1" pad="28"/>
+<contactref element="J52" pad="27"/>
+<contactref element="J52" pad="28"/>
 <contactref element="J51" pad="7"/>
 <wire x1="26.67" y1="-12.7" x2="26.67" y2="-10.16" width="1.016" layer="16"/>
@@
 </signal>
 <signal name="SENSORS_SDA">
-<contactref element="JP1" pad="1"/>
-<contactref element="JP1" pad="2"/>
+<contactref element="J52" pad="1"/>
+<contactref element="J52" pad="2"/>
 <contactref element="J50" pad="1"/>
 <contactref element="J1" pad="P1"/>
@@
 <signal name="SENSORS_SCL">
 <contactref element="J2" pad="P1"/>
-<contactref element="JP1" pad="3"/>
-<contactref element="JP1" pad="4"/>
+<contactref element="J52" pad="3"/>
+<contactref element="J52" pad="4"/>
 <contactref element="J50" pad="2"/>
 <wire x1="-3.81" y1="-10.16" x2="-3.81" y2="-12.7" width="1.016" layer="16"/>
@@
 <signal name="NRF_CTS">
 <contactref element="J3" pad="P1"/>
-<contactref element="JP1" pad="7"/>
-<contactref element="JP1" pad="8"/>
+<contactref element="J52" pad="7"/>
+<contactref element="J52" pad="8"/>
 <contactref element="J50" pad="4"/>
 <wire x1="1.27" y1="-12.7" x2="1.27" y2="-10.16" width="1.016" layer="16"/>
@@
 <signal name="NRF_RTS">
 <contactref element="J4" pad="P1"/>
-<contactref element="JP1" pad="9"/>
-<contactref element="JP1" pad="10"/>
+<contactref element="J52" pad="9"/>
+<contactref element="J52" pad="10"/>
 <contactref element="J50" pad="5"/>
 <wire x1="3.81" y1="-18.542" x2="3.81" y2="-12.7" width="1.016" layer="16"/>
@@
 <signal name="NRF_INT">
 <contactref element="J5" pad="P1"/>
-<contactref element="JP1" pad="11"/>
-<contactref element="JP1" pad="12"/>
+<contactref element="J52" pad="11"/>
+<contactref element="J52" pad="12"/>
 <contactref element="J50" pad="6"/>
 <wire x1="6.35" y1="-12.7" x2="6.35" y2="-10.16" width="1.016" layer="16"/>
@@
 <signal name="NRF_OUT">
 <contactref element="J6" pad="P1"/>
-<contactref element="JP1" pad="13"/>
-<contactref element="JP1" pad="14"/>
+<contactref element="J52" pad="13"/>
+<contactref element="J52" pad="14"/>
 <contactref element="J50" pad="7"/>
 <wire x1="8.89" y1="-18.542" x2="8.89" y2="-12.7" width="1.016" layer="16"/>
@@
 <signal name="NRF_IN">
 <contactref element="J7" pad="P1"/>
-<contactref element="JP1" pad="15"/>
-<contactref element="JP1" pad="16"/>
+<contactref element="J52" pad="15"/>
+<contactref element="J52" pad="16"/>
 <contactref element="J51" pad="1"/>
 <wire x1="11.43" y1="-12.7" x2="11.43" y2="-10.16" width="1.016" layer="16"/>
@@
 <signal name="!FTDI_RTS">
 <contactref element="J8" pad="P1"/>
-<contactref element="JP1" pad="17"/>
-<contactref element="JP1" pad="18"/>
+<contactref element="J52" pad="17"/>
+<contactref element="J52" pad="18"/>
 <contactref element="J51" pad="2"/>
 <wire x1="13.97" y1="-12.7" x2="13.97" y2="-18.542" width="1.016" layer="16"/>
@@
 <signal name="FTDI_IN">
 <contactref element="J9" pad="P1"/>
-<contactref element="JP1" pad="19"/>
-<contactref element="JP1" pad="20"/>
+<contactref element="J52" pad="19"/>
+<contactref element="J52" pad="20"/>
 <contactref element="J51" pad="3"/>
 <wire x1="16.51" y1="-12.7" x2="16.51" y2="-10.16" width="1.016" layer="16"/>
@@
 <signal name="FTDI_OUT">
 <contactref element="J10" pad="P1"/>
-<contactref element="JP1" pad="21"/>
-<contactref element="JP1" pad="22"/>
+<contactref element="J52" pad="21"/>
+<contactref element="J52" pad="22"/>
 <contactref element="J51" pad="4"/>
 <wire x1="19.05" y1="-18.542" x2="19.05" y2="-12.7" width="1.016" layer="16"/>
@@
 <signal name="ACC_INT1">
 <contactref element="J11" pad="P1"/>
-<contactref element="JP1" pad="23"/>
-<contactref element="JP1" pad="24"/>
+<contactref element="J52" pad="23"/>
+<contactref element="J52" pad="24"/>
 <contactref element="J51" pad="5"/>
 <wire x1="21.59" y1="-12.7" x2="21.59" y2="-10.16" width="1.016" layer="16"/>
@@
 <signal name="ACC_INT2">
 <contactref element="J12" pad="P1"/>
-<contactref element="JP1" pad="25"/>
-<contactref element="JP1" pad="26"/>
+<contactref element="J52" pad="25"/>
+<contactref element="J52" pad="26"/>
 <contactref element="J51" pad="6"/>
 <wire x1="24.13" y1="-18.542" x2="24.13" y2="-12.7" width="1.016" layer="16"/>
@@
 <contactref element="J39" pad="P1"/>
 <contactref element="J44" pad="2"/>
-<contactref element="JP1" pad="5"/>
-<contactref element="JP1" pad="6"/>
+<contactref element="J52" pad="5"/>
+<contactref element="J52" pad="6"/>
 <contactref element="J50" pad="3"/>
 <wire x1="-1.27" y1="-18.542" x2="-1.27" y2="-12.7" width="1.016" layer="16"/>

Commit message: updates to debug board
Parts:
- removed J52: (no value), pinhead:2X14
- added J45: (no value), pinhead:2X12
- J1, J10, J11, J12, J13, J2, J3, J4, J5, J6, J7, J8, J9: value MILLMAX_0985-X-15-20-71-14-11-0 -> MILLMAX_0908-X-15-20-75-14-11-0; device headers:POGO_0985-X-15-20-71-14-11-0 -> headers:POGO_0908-X-15-20-75-14-11-0
- J25, J26, J27, J28, J29, J30, J31, J32, J33, J34, J35, J36, J37: value MILLMAX_0908-X-15-20-75-14-11-0 -> MILLMAX_0985-X-15-20-71-14-11-0; device headers:POGO_0908-X-15-20-75-14-11-0 -> headers:POGO_0985-X-15-20-71-14-11-0
- J44: value TC2030-JLINK-L -> (none); device connector:TC2030-IDC -> pinhead:2X12
- J46: value SCREW_TERMINAL_12_0.100 -> (none); device headers:CONN_BLOCK_12 -> pinhead:2X14
- J47: value SCREW_TERMINAL_12_0.100 -> SCREW-TERMINAL_7_0.100; device headers:CONN_BLOCK_12 -> headers:CONN_BLOCK_7
- J48: value (none) -> SCREW-TERMINAL_7_0.100; device pinhead:2X12 -> headers:CONN_BLOCK_7
- J49: value (none) -> SCREW_TERMINAL_12_0.100; device pinhead:2X12 -> headers:CONN_BLOCK_12
- J50: value SCREW-TERMINAL_7_0.100 -> SCREW_TERMINAL_12_0.100; device headers:CONN_BLOCK_7 -> headers:CONN_BLOCK_12
- J51: value SCREW-TERMINAL_7_0.100 -> TC2030-JLINK-L; device headers:CONN_BLOCK_7 -> connector:TC2030-IDC
- moved J47 51.7 mm to (1.27, -18.5), turned to 0 degrees
- moved J50 51.7 mm to (37.6, 18.3), turned to 90 degrees
- moved J49 47.8 mm to (-17.3, 18.3)
- moved J48 47.0 mm to (19.1, -18.5), turned to 0 degrees
- moved J46 40.4 mm to (10.2, -11.4), turned to 0 degrees
- moved J51 35.7 mm to (-14.0, -5.08)
- moved J25 31.4 mm to (14.0, 33.0)
- moved J12 26.9 mm to (1.27, 4.32)
- moved J44 23.7 mm to (-10.2, 18.3), turned to 270 degrees
- moved J11 21.7 mm to (1.27, 6.86)
- moved J36 20.9 mm to (15.1, 27.4)
- moved J13 20.9 mm to (19.1, 32.3)
- moved J10 20.2 mm to (1.27, 9.40)
- moved J34 19.5 mm to (8.46, 28.3)
- moved J14 18.0 mm to (19.1, 29.7)
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Connections:
- net !FTDI_RTS: now also J32.P1, J46.17, J46.18, J48.2; no longer J51.2, J52.17, J52.18, J8.P1
- net !LIGHT_INT: now also J37.P1, J46.27, J46.28, J48.7; no longer J13.P1, J51.7, J52.27, J52.28
- net !NRF_RESET: now also J51.3; no longer J44.3
- net 3V3: now also J13.P$1, J45.1, J45.2, J50.12; no longer J26.P$1, J47.12, J49.1, J49.2
- net A0: now also J12.P$1, J44.23, J44.24, J49.12; no longer J25.P$1, J46.12, J48.23, J48.24
- net A1: now also J11.P$1, J44.21, J44.22, J49.11; no longer J24.P$1, J46.11, J48.21, J48.22
- net A2: now also J10.P$1, J44.19, J44.20, J49.10; no longer J23.P$1, J46.10, J48.19, J48.20
- net A3: now also J44.17, J44.18, J49.9, J9.P$1; no longer J22.P$1, J46.9, J48.17, J48.18
- net A4: now also J44.15, J44.16, J49.8, J8.P$1; no longer J21.P$1, J46.8, J48.15, J48.16
- net A5: now also J44.13, J44.14, J49.7, J7.P$1; no longer J20.P$1, J46.7, J48.13, J48.14
- net ACC_INT1: now also J35.P1, J46.23, J46.24, J48.5; no longer J11.P1, J51.5, J52.23, J52.24
- net ACC_INT2: now also J36.P1, J46.25, J46.26, J48.6; no longer J12.P1, J51.6, J52.25, J52.26
- net D0: now also J24.P$1, J45.23, J45.24, J50.1; no longer J37.P$1, J47.1, J49.23, J49.24
- net D1: now also J23.P$1, J45.21, J45.22, J50.2; no longer J36.P$1, J47.2, J49.21, J49.22
- net D2: now also J22.P$1, J45.19, J45.20, J50.3; no longer J35.P$1, J47.3, J49.19, J49.20
- net D3: now also J21.P$1, J45.17, J45.18, J50.4; no longer J34.P$1, J47.4, J49.17, J49.18
- net D4: now also J20.P$1, J45.15, J45.16, J50.5; no longer J33.P$1, J47.5, J49.15, J49.16
- net D5: now also J19.P$1, J45.13, J45.14, J50.6; no longer J32.P$1, J47.6, J49.13, J49.14
- net D6: now also J18.P$1, J45.11, J45.12, J50.7; no longer J31.P$1, J47.7, J49.11, J49.12
- net D7: now also J17.P$1, J45.10, J45.9, J50.8; no longer J30.P$1, J47.8, J49.10, J49.9
- net DAC: now also J44.11, J44.12, J49.6, J6.P$1; no longer J19.P$1, J46.6, J48.11, J48.12
- net FTDI_IN: now also J33.P1, J46.19, J46.20, J48.3; no longer J51.3, J52.19, J52.20, J9.P1
- net FTDI_OUT: now also J34.P1, J46.21, J46.22, J48.4; no longer J10.P1, J51.4, J52.21, J52.22
- net GND: now also J16.P$1, J2.P$1, J43.P1, J44.3, J44.4, J45.7, J45.8, J49.2, J50.9, J51.5; no longer J15.P$1, J29.P$1, J42.P1, J44.5, J46.2, J47.9, J48.3, J48.4, J49.7, J49.8
- net NRF_CTS: now also J27.P1, J46.7, J46.8, J47.4; no longer J3.P1, J50.4, J52.7, J52.8
- net NRF_IN: now also J31.P1, J46.15, J46.16, J48.1; no longer J51.1, J52.15, J52.16, J7.P1
- net NRF_INT: now also J29.P1, J46.11, J46.12, J47.6; no longer J5.P1, J50.6, J52.11, J52.12
- net NRF_OUT: now also J30.P1, J46.13, J46.14, J47.7; no longer J50.7, J52.13, J52.14, J6.P1
- net NRF_RTS: now also J28.P1, J46.10, J46.9, J47.5; no longer J4.P1, J50.5, J52.10, J52.9
- net NRF_SWDCLK: now also J51.4; no longer J44.4
- net NRF_SWDIO: now also J46.5, J46.6, J47.3, J51.2; no longer J44.2, J50.3, J52.5, J52.6
- net NRF_SWO: now also J42.P1; no longer J43.P1
- net NRV_VCC: now also J51.1; no longer J44.1
- net RST: now also J14.P$1, J45.3, J45.4, J50.11; no longer J27.P$1, J47.11, J49.3, J49.4
- net RX: now also J4.P$1, J44.7, J44.8, J49.4; no longer J17.P$1, J46.4, J48.7, J48.8
- net SENSORS_SCL: now also J26.P1, J46.3, J46.4, J47.2; no longer J2.P1, J50.2, J52.3, J52.4
- net SENSORS_SDA: now also J25.P1, J46.1, J46.2, J47.1; no longer J1.P1, J50.1, J52.1, J52.2
- net TX: now also J3.P$1, J44.5, J44.6, J49.3; no longer J16.P$1, J46.3, J48.5, J48.6
- net VBAT: now also J15.P$1, J45.5, J45.6, J50.10; no longer J28.P$1, J47.10, J49.5, J49.6
- net VIN: now also J1.P$1, J44.1, J44.2, J49.1; no longer J14.P$1, J46.1, J48.1, J48.2
- net WKP: now also J44.10, J44.9, J49.5, J5.P$1; no longer J18.P$1, J46.5, J48.10, J48.9
