File: hardware/hail-debug/rev_a/hail-debug.sch (EAGLE design)
At the start: 58 parts, among them J1 MILLMAX_0985-X-15-20-71-14-11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, J10 MILLMAX_0985-X-15-20-71-14-11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, J11 MILLMAX_0985-X-15-20-71-14-11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, J12 MILLMAX_0985-X-15-20-71-14-11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, J13 MILLMAX_0985-X-15-20-71-14-11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, J14 MILLMAX_0908-X-15-20-75-14-11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, J15 MILLMAX_0908-X-15-20-75-14-11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, J16 MILLMAX_0908-X-15-20-75-14-11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, J17 MILLMAX_0908-X-15-20-75-14-11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, J18 MILLMAX_0908-X-15-20-75-14-11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, J19 MILLMAX_0908-X-15-20-75-14-11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, J2 MILLMAX_0985-X-15-20-71-14-11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, J20 MILLMAX_0908-X-15-20-75-14-11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, J21 MILLMAX_0908-X-15-20-75-14-11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, J22 MILLMAX_0908-X-15-20-75-14-11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, J23 MILLMAX_0908-X-15-20-75-14-11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, J24 MILLMAX_0908-X-15-20-75-14-11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, J25 MILLMAX_0908-X-15-20-75-14-11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, J26 MILLMAX_0908-X-15-20-75-14-11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, J27 MILLMAX_0908-X-15-20-75-14-11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, J28 MILLMAX_0908-X-15-20-75-14-11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, J29 MILLMAX_0908-X-15-20-75-14-11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, J3 MILLMAX_0985-X-15-20-71-14-11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, J30 MILLMAX_0908-X-15-20-75-14-11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, J31 MILLMAX_0908-X-15-20-75-14-11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, J32 MILLMAX_0908-X-15-20-75-14-11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, J33 MILLMAX_0908-X-15-20-75-14-11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, J34 MILLMAX_0908-X-15-20-75-14-11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, J35 MILLMAX_0908-X-15-20-75-14-11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, J36 MILLMAX_0908-X-15-20-75-14-11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, J37 MILLMAX_0908-X-15-20-75-14-11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, J38 MILLMAX_0985-X-15-20-71-14-11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, J39 MILLMAX_0985-X-15-20-71-14-11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, J4 MILLMAX_0985-X-15-20-71-14-11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, J40 MILLMAX_0985-X-15-20-71-14-11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, J41 MILLMAX_0985-X-15-20-71-14-11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, J42 MILLMAX_0985-X-15-20-71-14-11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, J43 MILLMAX_0985-X-15-20-71-14-11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, J44 TC2030-JLINK-L, J46 SCREW_TERMINAL_12_0.100, J47 SCREW_TERMINAL_12_0.100, J5 MILLMAX_0985-X-15-20-71-14-11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, J50 SCREW-TERMINAL_7_0.100, J51 SCREW-TERMINAL_7_0.100, J6 MILLMAX_0985-X-15-20-71-14-11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, J7 MILLMAX_0985-X-15-20-71-14-11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, J8 MILLMAX_0985-X-15-20-71-14-11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, J9 MILLMAX_0985-X-15-20-71-14-11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

Commit message: small fixes
Parts:
- renumbered JP1 to J52
Other:
- moved on the sheet: H1, H2, H3, H4, H5
Changed lines of the file:
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@@
 <schematic xreflabel="%F%N/%S.%C%R" xrefpart="/%S.%C%R">
 <attributes>
+<attribute name="AUTHOR" value="Brad Campbell"/>
+<attribute name="REV" value="A"/>
+<attribute name="TITLE" value="Hail Debug Board"/>
 </attributes>
 <variantdefs>
@@
 <part name="H3" library="holes" deviceset="MOUNT-HOLE" device="3.2"/>
 <part name="H4" library="holes" deviceset="MOUNT-HOLE" device="3.2"/>
-<part name="JP1" library="pinhead" deviceset="PINHD-2X14" device=""/>
+<part name="J52" library="pinhead" deviceset="PINHD-2X14" device=""/>
 <part name="J50" library="headers" deviceset="SCREW-TERMINAL_7_0.100" device=""/>
 <part name="J51" library="headers" deviceset="SCREW-TERMINAL_7_0.100" device=""/>
@@
 <instance part="J44" gate="G$1" x="203.2" y="152.4"/>
 <instance part="J48" gate="A" x="124.46" y="99.06"/>
-<instance part="J46" gate="G$1" x="149.86" y="99.06" rot="MR0"/>
+<instance part="J46" gate="G$1" x="149.86" y="99.06" smashed="yes" rot="MR0">
+<attribute name="NAME" x="154.94" y="114.808" size="1.778" layer="95" rot="MR0"/>
+<attribute name="VALUE" x="160.02" y="114.3" size="1.778" layer="96" rot="MR270"/>
+</instance>
 <instance part="J49" gate="A" x="124.46" y="55.88"/>
-<instance part="J47" gate="G$1" x="149.86" y="53.34" rot="R180"/>
-<instance part="H1" gate="G$1" x="99.06" y="10.16"/>
-<instance part="H2" gate="G$1" x="99.06" y="15.24"/>
-<instance part="H3" gate="G$1" x="99.06" y="20.32"/>
-<instance part="H4" gate="G$1" x="99.06" y="25.4"/>
-<instance part="JP1" gate="A" x="139.7" y="149.86"/>
+<instance part="J47" gate="G$1" x="149.86" y="53.34" smashed="yes" rot="R180">
+<attribute name="NAME" x="154.94" y="37.592" size="1.778" layer="95" rot="R180"/>
+<attribute name="VALUE" x="160.02" y="35.56" size="1.778" layer="96" rot="R90"/>
+</instance>
+<instance part="H1" gate="G$1" x="228.6" y="25.4"/>
+<instance part="H2" gate="G$1" x="228.6" y="30.48"/>
+<instance part="H3" gate="G$1" x="228.6" y="35.56"/>
+<instance part="H4" gate="G$1" x="228.6" y="40.64"/>
+<instance part="J52" gate="A" x="139.7" y="149.86"/>
 <instance part="J50" gate="G$1" x="160.02" y="157.48" smashed="yes" rot="MR0">
 <attribute name="NAME" x="162.56" y="170.18" size="1.27" layer="95" rot="MR0"/>
@@
 <attribute name="NAME" x="162.56" y="152.4" size="1.27" layer="95" rot="MR0"/>
 </instance>
-<instance part="H5" gate="G$1" x="99.06" y="30.48"/>
+<instance part="H5" gate="G$1" x="228.6" y="45.72"/>
 <instance part="S1" gate="G$1" x="208.28" y="93.98"/>
 <instance part="LOGO1" gate="G$1" x="236.22" y="177.8"/>
@@
 <wire x1="17.78" y1="132.08" x2="137.16" y2="132.08" width="0.1524" layer="91"/>
 <label x="157.48" y="132.08" size="1.27" layer="95" xref="yes"/>
-<pinref part="JP1" gate="A" pin="27"/>
-<pinref part="JP1" gate="A" pin="28"/>
+<pinref part="J52" gate="A" pin="27"/>
+<pinref part="J52" gate="A" pin="28"/>
 <wire x1="144.78" y1="132.08" x2="137.16" y2="132.08" width="0.1524" layer="91"/>
 <junction x="137.16" y="132.08"/>
@@
 <segment>
 <label x="157.48" y="165.1" size="1.27" layer="95" xref="yes"/>
-<pinref part="JP1" gate="A" pin="1"/>
+<pinref part="J52" gate="A" pin="1"/>
 <wire x1="129.54" y1="165.1" x2="137.16" y2="165.1" width="0.1524" layer="91"/>
-<pinref part="JP1" gate="A" pin="2"/>
+<pinref part="J52" gate="A" pin="2"/>
 <wire x1="144.78" y1="165.1" x2="137.16" y2="165.1" width="0.1524" layer="91"/>
 <junction x="137.16" y="165.1"/>
@@
 <label x="157.48" y="162.56" size="1.27" layer="95" xref="yes"/>
 <wire x1="132.08" y1="160.02" x2="132.08" y2="162.56" width="0.1524" layer="91"/>
-<pinref part="JP1" gate="A" pin="3"/>
+<pinref part="J52" gate="A" pin="3"/>
 <wire x1="132.08" y1="162.56" x2="137.16" y2="162.56" width="0.1524" layer="91"/>
-<pinref part="JP1" gate="A" pin="4"/>
+<pinref part="J52" gate="A" pin="4"/>
 <wire x1="144.78" y1="162.56" x2="137.16" y2="162.56" width="0.1524" layer="91"/>
 <junction x="137.16" y="162.56"/>
@@
 <wire x1="93.98" y1="160.02" x2="93.98" y2="157.48" width="0.1524" layer="91"/>
 <label x="157.48" y="157.48" size="1.27" layer="95" xref="yes"/>
-<pinref part="JP1" gate="A" pin="7"/>
+<pinref part="J52" gate="A" pin="7"/>
 <wire x1="93.98" y1="157.48" x2="137.16" y2="157.48" width="0.1524" layer="91"/>
-<pinref part="JP1" gate="A" pin="8"/>
+<pinref part="J52" gate="A" pin="8"/>
 <wire x1="137.16" y1="157.48" x2="144.78" y2="157.48" width="0.1524" layer="91"/>
 <junction x="137.16" y="157.48"/>
@@
 <wire x1="86.36" y1="157.48" x2="86.36" y2="154.94" width="0.1524" layer="91"/>
 <label x="157.48" y="154.94" size="1.27" layer="95" xref="yes"/>
-<pinref part="JP1" gate="A" pin="9"/>
+<pinref part="J52" gate="A" pin="9"/>
 <wire x1="86.36" y1="154.94" x2="137.16" y2="154.94" width="0.1524" layer="91"/>
-<pinref part="JP1" gate="A" pin="10"/>
+<pinref part="J52" gate="A" pin="10"/>
 <wire x1="144.78" y1="154.94" x2="137.16" y2="154.94" width="0.1524" layer="91"/>
 <junction x="137.16" y="154.94"/>
@@
 <wire x1="78.74" y1="152.4" x2="137.16" y2="152.4" width="0.1524" layer="91"/>
 <label x="157.48" y="152.4" size="1.27" layer="95" xref="yes"/>
-<pinref part="JP1" gate="A" pin="11"/>
-<pinref part="JP1" gate="A" pin="12"/>
+<pinref part="J52" gate="A" pin="11"/>
+<pinref part="J52" gate="A" pin="12"/>
 <wire x1="137.16" y1="152.4" x2="144.78" y2="152.4" width="0.1524" layer="91"/>
 <junction x="137.16" y="152.4"/>
@@
 <wire x1="71.12" y1="149.86" x2="137.16" y2="149.86" width="0.1524" layer="91"/>
 <label x="157.48" y="149.86" size="1.27" layer="95" xref="yes"/>
-<pinref part="JP1" gate="A" pin="13"/>
-<pinref part="JP1" gate="A" pin="14"/>
+<pinref part="J52" gate="A" pin="13"/>
+<pinref part="J52" gate="A" pin="14"/>
 <wire x1="144.78" y1="149.86" x2="137.16" y2="149.86" width="0.1524" layer="91"/>
 <junction x="137.16" y="149.86"/>
@@
 <wire x1="63.5" y1="147.32" x2="137.16" y2="147.32" width="0.1524" layer="91"/>
 <label x="157.48" y="147.32" size="1.27" layer="95" xref="yes"/>
-<pinref part="JP1" gate="A" pin="15"/>
-<pinref part="JP1" gate="A" pin="16"/>
+<pinref part="J52" gate="A" pin="15"/>
+<pinref part="J52" gate="A" pin="16"/>
 <wire x1="137.16" y1="147.32" x2="144.78" y2="147.32" width="0.1524" layer="91"/>
 <junction x="137.16" y="147.32"/>
@@
 <wire x1="55.88" y1="144.78" x2="137.16" y2="144.78" width="0.1524" layer="91"/>
 <label x="157.48" y="144.78" size="1.27" layer="95" xref="yes"/>
-<pinref part="JP1" gate="A" pin="17"/>
-<pinref part="JP1" gate="A" pin="18"/>
+<pinref part="J52" gate="A" pin="17"/>
+<pinref part="J52" gate="A" pin="18"/>
 <wire x1="144.78" y1="144.78" x2="137.16" y2="144.78" width="0.1524" layer="91"/>
 <junction x="137.16" y="144.78"/>
@@
 <wire x1="48.26" y1="142.24" x2="137.16" y2="142.24" width="0.1524" layer="91"/>
 <label x="157.48" y="142.24" size="1.27" layer="95" xref="yes"/>
-<pinref part="JP1" gate="A" pin="19"/>
-<pinref part="JP1" gate="A" pin="20"/>
+<pinref part="J52" gate="A" pin="19"/>
+<pinref part="J52" gate="A" pin="20"/>
 <wire x1="137.16" y1="142.24" x2="144.78" y2="142.24" width="0.1524" layer="91"/>
 <junction x="137.16" y="142.24"/>
@@
 <wire x1="40.64" y1="139.7" x2="137.16" y2="139.7" width="0.1524" layer="91"/>
 <label x="157.48" y="139.7" size="1.27" layer="95" xref="yes"/>
-<pinref part="JP1" gate="A" pin="21"/>
-<pinref part="JP1" gate="A" pin="22"/>
+<pinref part="J52" gate="A" pin="21"/>
+<pinref part="J52" gate="A" pin="22"/>
 <wire x1="137.16" y1="139.7" x2="144.78" y2="139.7" width="0.1524" layer="91"/>
 <junction x="137.16" y="139.7"/>
@@
 <wire x1="33.02" y1="137.16" x2="137.16" y2="137.16" width="0.1524" layer="91"/>
 <label x="157.48" y="137.16" size="1.27" layer="95" xref="yes"/>
-<pinref part="JP1" gate="A" pin="23"/>
-<pinref part="JP1" gate="A" pin="24"/>
+<pinref part="J52" gate="A" pin="23"/>
+<pinref part="J52" gate="A" pin="24"/>
 <wire x1="144.78" y1="137.16" x2="137.16" y2="137.16" width="0.1524" layer="91"/>
 <junction x="137.16" y="137.16"/>
@@
 <wire x1="25.4" y1="134.62" x2="137.16" y2="134.62" width="0.1524" layer="91"/>
 <label x="157.48" y="134.62" size="1.27" layer="95" xref="yes"/>
-<pinref part="JP1" gate="A" pin="25"/>
-<pinref part="JP1" gate="A" pin="26"/>
+<pinref part="J52" gate="A" pin="25"/>
+<pinref part="J52" gate="A" pin="26"/>
 <wire x1="137.16" y1="134.62" x2="144.78" y2="134.62" width="0.1524" layer="91"/>
 <junction x="137.16" y="134.62"/>
@@
 </segment>
 <segment>
-<pinref part="JP1" gate="A" pin="5"/>
-<pinref part="JP1" gate="A" pin="6"/>
+<pinref part="J52" gate="A" pin="5"/>
+<pinref part="J52" gate="A" pin="6"/>
 <wire x1="137.16" y1="160.02" x2="144.78" y2="160.02" width="0.1524" layer="91"/>
 <wire x1="144.78" y1="160.02" x2="152.4" y2="160.02" width="0.1524" layer="91"/>

Commit message: updates to debug board
Parts:
- removed J52: (no value), pinhead:PINHD-2X14
- added J45: (no value), pinhead:PINHD-2X12
- J1, J10, J11, J12, J13, J2, J3, J4, J5, J6, J7, J8, J9: value MILLMAX_0985-X-15-20-71-14-11-0 -> MILLMAX_0908-X-15-20-75-14-11-0; device headers:MILLMAX_0985-X-15-20-71-14-11-0 -> headers:MILLMAX_0908-X-15-20-75-14-11-0
- J25, J26, J27, J28, J29, J30, J31, J32, J33, J34, J35, J36, J37: value MILLMAX_0908-X-15-20-75-14-11-0 -> MILLMAX_0985-X-15-20-71-14-11-0; device headers:MILLMAX_0908-X-15-20-75-14-11-0 -> headers:MILLMAX_0985-X-15-20-71-14-11-0
- J44: value TC2030-JLINK-L -> (none); device connector:TC2030-JLINK-L -> pinhead:PINHD-2X12; DIGIKEY (none) -> S2011EC-12-ND
- J46: value SCREW_TERMINAL_12_0.100 -> (none); device headers:SCREW_TERMINAL_12_0.100 -> pinhead:PINHD-2X14; DIGIKEY (none) -> S2011EC-14-ND
- J47: value SCREW_TERMINAL_12_0.100 -> SCREW-TERMINAL_7_0.100; device headers:SCREW_TERMINAL_12_0.100 -> headers:SCREW-TERMINAL_7_0.100
- J48: value (none) -> SCREW-TERMINAL_7_0.100; device pinhead:PINHD-2X12 -> headers:SCREW-TERMINAL_7_0.100
- J49: value (none) -> SCREW_TERMINAL_12_0.100; device pinhead:PINHD-2X12 -> headers:SCREW_TERMINAL_12_0.100
- J50: value SCREW-TERMINAL_7_0.100 -> SCREW_TERMINAL_12_0.100; device headers:SCREW-TERMINAL_7_0.100 -> headers:SCREW_TERMINAL_12_0.100
- J51: value SCREW-TERMINAL_7_0.100 -> TC2030-JLINK-L; device headers:SCREW-TERMINAL_7_0.100 -> connector:TC2030-JLINK-L
Connections:
- net !FTDI_RTS: now also J32.P$1, J46.17, J46.18, J48.2; no longer J51.2, J52.17, J52.18, J8.P$1
- net !LIGHT_INT: now also J37.P$1, J46.27, J46.28, J48.7; no longer J13.P$1, J51.7, J52.27, J52.28
- net !NRF_RESET: now also J51.!RESET; no longer J44.!RESET
- net 3V3: now also J13.P$1, J45.1, J45.2, J50.12; no longer J26.P$1, J47.12, J49.1, J49.2
- net A0: now also J12.P$1, J44.23, J44.24, J49.12; no longer J25.P$1, J46.12, J48.23, J48.24
- net A1: now also J11.P$1, J44.21, J44.22, J49.11; no longer J24.P$1, J46.11, J48.21, J48.22
- net A2: now also J10.P$1, J44.19, J44.20, J49.10; no longer J23.P$1, J46.10, J48.19, J48.20
- net A3: now also J44.17, J44.18, J49.9, J9.P$1; no longer J22.P$1, J46.9, J48.17, J48.18
- net A4: now also J44.15, J44.16, J49.8, J8.P$1; no longer J21.P$1, J46.8, J48.15, J48.16
- net A5: now also J44.13, J44.14, J49.7, J7.P$1; no longer J20.P$1, J46.7, J48.13, J48.14
- net ACC_INT1: now also J35.P$1, J46.23, J46.24, J48.5; no longer J11.P$1, J51.5, J52.23, J52.24
- net ACC_INT2: now also J36.P$1, J46.25, J46.26, J48.6; no longer J12.P$1, J51.6, J52.25, J52.26
- net D0: now also J24.P$1, J45.23, J45.24, J50.1; no longer J37.P$1, J47.1, J49.23, J49.24
- net D1: now also J23.P$1, J45.21, J45.22, J50.2; no longer J36.P$1, J47.2, J49.21, J49.22
- net D2: now also J22.P$1, J45.19, J45.20, J50.3; no longer J35.P$1, J47.3, J49.19, J49.20
- net D3: now also J21.P$1, J45.17, J45.18, J50.4; no longer J34.P$1, J47.4, J49.17, J49.18
- net D4: now also J20.P$1, J45.15, J45.16, J50.5; no longer J33.P$1, J47.5, J49.15, J49.16
- net D5: now also J19.P$1, J45.13, J45.14, J50.6; no longer J32.P$1, J47.6, J49.13, J49.14
- net D6: now also J18.P$1, J45.11, J45.12, J50.7; no longer J31.P$1, J47.7, J49.11, J49.12
- net D7: now also J17.P$1, J45.10, J45.9, J50.8; no longer J30.P$1, J47.8, J49.10, J49.9
- net DAC: now also J44.11, J44.12, J49.6, J6.P$1; no longer J19.P$1, J46.6, J48.11, J48.12
- net FTDI_IN: now also J33.P$1, J46.19, J46.20, J48.3; no longer J51.3, J52.19, J52.20, J9.P$1
- net FTDI_OUT: now also J34.P$1, J46.21, J46.22, J48.4; no longer J10.P$1, J51.4, J52.21, J52.22
- net GND: now also J16.P$1, J2.P$1, J43.P$1, J44.3, J44.4, J45.7, J45.8, J49.2, J50.9, J51.GND; no longer J15.P$1, J29.P$1, J42.P$1, J44.GND, J46.2, J47.9, J48.3, J48.4, J49.7, J49.8
- net NRF_CTS: now also J27.P$1, J46.7, J46.8, J47.4; no longer J3.P$1, J50.4, J52.7, J52.8
- net NRF_IN: now also J31.P$1, J46.15, J46.16, J48.1; no longer J51.1, J52.15, J52.16, J7.P$1
- net NRF_INT: now also J29.P$1, J46.11, J46.12, J47.6; no longer J5.P$1, J50.6, J52.11, J52.12
- net NRF_OUT: now also J30.P$1, J46.13, J46.14, J47.7; no longer J50.7, J52.13, J52.14, J6.P$1
- net NRF_RTS: now also J28.P$1, J46.10, J46.9, J47.5; no longer J4.P$1, J50.5, J52.10, J52.9
- net NRF_SWDCLK: now also J51.SWDCLK; no longer J44.SWDCLK
- net NRF_SWDIO: now also J46.5, J46.6, J47.3, J51.SWDIO; no longer J44.SWDIO, J50.3, J52.5, J52.6
- net NRF_SWO: now also J42.P$1; no longer J43.P$1
- net NRV_VCC: now also J51.VCC; no longer J44.VCC
- net RST: now also J14.P$1, J45.3, J45.4, J50.11; no longer J27.P$1, J47.11, J49.3, J49.4
- net RX: now also J4.P$1, J44.7, J44.8, J49.4; no longer J17.P$1, J46.4, J48.7, J48.8
- net SENSORS_SCL: now also J26.P$1, J46.3, J46.4, J47.2; no longer J2.P$1, J50.2, J52.3, J52.4
- net SENSORS_SDA: now also J25.P$1, J46.1, J46.2, J47.1; no longer J1.P$1, J50.1, J52.1, J52.2
- net TX: now also J3.P$1, J44.5, J44.6, J49.3; no longer J16.P$1, J46.3, J48.5, J48.6
- net VBAT: now also J15.P$1, J45.5, J45.6, J50.10; no longer J28.P$1, J47.10, J49.5, J49.6
- net VIN: now also J1.P$1, J44.1, J44.2, J49.1; no longer J14.P$1, J46.1, J48.1, J48.2
- net WKP: now also J44.10, J44.9, J49.5, J5.P$1; no longer J18.P$1, J46.5, J48.10, J48.9
Other:
- moved on the sheet: J1, J10, J11, J12, J13, J14, J15, J16, J17, J18, J19, J2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
