File: hardware/hail/rev_b/hail.sch (EAGLE design)
At the start: 73 parts, among them J1 MICRO_USB_B_HIROSE_ZX62R-B-5P, J2 TC2030-JLINK-NL_NOSILK, J3 TC2030-JLINK-NL_NOSILK, U1 FT231XQ, U2 FXOS8700CQ, U3 ISL29035, U4 MAX8887EZK33+T, U5 NRF51822QF, U6 SAM4LC8BA, U7 SI7021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

Commit message: Hail rev B!
Parts:
- removed JP3: M12PTH-CST-L, Particle:M12PTH-CST-L
- removed JP4: M12PTH-CST-R, Particle:M12PTH-CST-R
- added J4, J5: TC2030-JLINK-NL_NOSILK, connector:TC2030-JLINK-NL_NOSILK
- J2: value TC2030-JLINK-NL_NOSILK -> M12PTH-CST-L; device connector:TC2030-JLINK-NL_NOSILK -> Particle:M12PTH-CST-L; DIGIKEY (none) -> S1011E-12-ND
- J3: value TC2030-JLINK-NL_NOSILK -> M12PTH-CST-R; device connector:TC2030-JLINK-NL_NOSILK -> Particle:M12PTH-CST-R; DIGIKEY (none) -> S1011E-12-ND
- R10: value 100k -> 10k; DIGIKEY 1276-3432-1-ND -> 1276-3431-1-ND
- R13: value 1k -> 100k; DIGIKEY 1276-3430-1-ND -> 1276-3432-1-ND
- R6: value 10k -> 1k; DIGIKEY 1276-3431-1-ND -> 1276-3430-1-ND
Connections:
- net !LIGHT_INT: now also R9.1; no longer R8.1
- net !NRF_RESET: now also J5.SWDIO; no longer J3.SWDIO
- net !SAM4L_RESET: now also J3.11, J4.!RESET, R6.2; no longer J2.!RESET, JP4.11, R13.2
- net 5V: now also J2.12; no longer JP3.12
- net BUCK/LDO_N1: now also R10.2; no longer R9.2
- net BUTTON: now also R13.1; no longer R12.1
- net GND: now also J2.11, J3.9, J4.GND, J5.GND, R10.1; no longer J2.GND, J3.GND, JP3.11, JP4.9, R9.1
- net N$24: now also R6.1; no longer R13.1
- net N$6: now also J5.SWDCLK; no longer J3.SWDCLK
- net PARTICLE_A0: now also J2.1; no longer JP3.1
- net PARTICLE_A1: now also J2.2; no longer JP3.2
- net PARTICLE_A2: now also J2.3; no longer JP3.3
- net PARTICLE_A3: now also J2.4; no longer JP3.4
- net PARTICLE_A4: now also J2.5; no longer JP3.5
- net PARTICLE_A5: now also J2.6; no longer JP3.6
- net PARTICLE_D0: now also J3.1; no longer JP4.1
- net PARTICLE_D1: now also J3.2; no longer JP4.2
- net PARTICLE_D2: now also J3.3; no longer JP4.3
- net PARTICLE_D3: now also J3.4; no longer JP4.4
- net PARTICLE_D4: now also J3.5; no longer JP4.5
- net PARTICLE_D5: now also J3.6; no longer JP4.6
- net PARTICLE_D6: now also J3.7; no longer JP4.7
- net PARTICLE_D7: now also J3.8; no longer JP4.8
- net PARTICLE_DAC: now also J2.7; no longer JP3.7
- net PARTICLE_RX: now also J2.9; no longer JP3.9
- net PARTICLE_TX: now also J2.10; no longer JP3.10
- net PARTICLE_WKP: now also J2.8; no longer JP3.8
- net SAM4L_SWDCLK: now also J4.SWDCLK, R12.1; no longer J2.SWDCLK, R11.1
- net SAM4L_SWDIO: now also J4.SWDIO, R11.1; no longer J2.SWDIO, R10.1
- net SENSORS_SCL: now also R8.1; no longer R7.1
- net SENSORS_SDA: now also R7.1; no longer R6.1
- net VCC: now also J3.12, J4.VCC, J5.VCC, R13.2, R9.2; no longer J2.VCC, J3.VCC, JP4.12, R10.2, R6.2
Other:
- moved on the sheet: R10, R11, R12, R7, R8

Commit message: add mpn
still more to be done here. if you add mpn for house parts you don't get
the house parts. macrofab is frustratingly difficult to set up. arg.
Parts:
- A1: MPN (none) -> FR05-S1-N-0110B
- B1: MPN (none) -> BAL-NRF01D3
- C1: MPN (none) -> GRM1555C1H1R5BA01D
- C10, C11, C12, C13, C14, C15, C16, C17, C18, C19, C20, C21, C22: MPN (none) -> GRM155R71A104JA01D
- C2, C3: MPN (none) -> GRM1555C1H8R0BA01D
- C23, C24, C25: MPN (none) -> ZRB15XR61A475KE01D
- C4, C5: MPN (none) -> GRM1555C1H120GA01D
- C6: MPN (none) -> GRM155R71H102KA01D
- C7: MPN (none) -> GRM155R71E222KA01D
- C8: MPN (none) -> GRM155R71H103JA88D
- C9: MPN (none) -> C1005X7R1C473K050BC
- D1: MPN (none) -> SML-LX0404SIUPGUSB
- FB1: MPN (none) -> CIM05J152NC
- J1: MPN (none) -> ZX62R-B-5P(30)
- J2, J3, J4, J5: POPULATE (none) -> 0
- L1: MPN (none) -> LQW15AN6N8G00D
- LED1: MPN (none) -> LTST-C194TBKT
- R1, R2, R3, R4, R5, R6: MPN (none) -> MF-RES-0402-1K; MPN1 (none) -> RC1005F102CS
- R10, R7, R8, R9: MPN (none) -> RC1005F103CS
- R11, R12, R13: MPN (none) -> RC1005F104CS
- S1, S2: MPN (none) -> B3U-1000P
- U4: MPN (none) -> MAX8887EZK33+T
- U5: MPN (none) -> NRF51822-QFAC-R7
- U6: MPN (none) -> ATSAM4LC8BA-MU
- U7: MPN (none) -> SI7021-A20-GM1
- X1: MPN (none) -> 8Y-16.000MAAV-T
- X2: MPN (none) -> FH1600015

Commit message: finally got the attributes right
Parts:
- C10, C11, C12, C13, C14, C15, C16, C17, C18, C19, C20, C21, C22: MPN GRM155R71A104JA01D -> MF-CAP-0402-0.1uF; MPN1 (none) -> GRM155R71A104JA01D
- C6: MPN GRM155R71H102KA01D -> MF-CAP-0402-1nF; MPN1 (none) -> GRM155R71H102KA01D
- C8: MPN GRM155R71H103JA88D -> MF-CAP-0402-0.01uF; MPN1 (none) -> GRM155R71H103JA88D
- J2, J3: MPN (none) -> MF-CON-2.54mm-01x12
- LED1: MPN LTST-C194TBKT -> MF-LED-0603-GREEN; MPN1 (none) -> LTST-C194TBKT
- R10, R7, R8, R9: MPN RC1005F103CS -> MF-RES-0402-10K; MPN1 (none) -> RC1005F103CS
- R11, R12, R13: MPN RC1005F104CS -> MF-RES-0402-100K; MPN1 (none) -> RC1005F104CS
