File: hardware/hail-wifi/rev_a/hail-wifi.brd (EAGLE design)
At the start: 20.3 x 55.9 mm, 20 parts, among them U1 ESP-WROOM-S2, U2 V_REG_LDOSMD, U3 PHOTON_WITH_HEADERS

Commit message: some updates to hail-wifi
Rev a doesn't work (wrong esp chip), but I hacked a version which I hope
will work and then I will make a rev b.
Parts:
- C1, C2: value 1uF -> 0.1uF
- C3: value 0.1uF -> 1uF
- C4: value 10uF -> 1uF
- C5: value 0.1uF -> 10uF
- moved C1 18.0 mm to (5.08, 31.5)
- moved C3 18.0 mm to (10.9, 14.5)
- moved C4 11.2 mm to (11.2, 20.6)
- moved C2 8.14 mm to (11.7, 28.7), turned to 270 degrees
- moved C5 6.73 mm to (5.08, 30.0), turned to 0 degrees
- moved U1 2.16 mm to (2.16, 34.8)
Connections:
- net +3V3: now also C1.1, C5.1; no longer C2.1, C3.1
- net 5V: now also C3.1; no longer C1.1
- net N$6: now also C2.1; no longer C5.1
Routing:
- net RST: track 52.2 -> 54.7 mm
- net TX: track 39.5 -> 41.7 mm
- net N$5: track 14.9 -> 17.1 mm
- net +3V3: track 63.1 -> 65.2 mm
- net MOSI: track 15.2 -> 17.3 mm
- net N$2: track 15.6 -> 17.7 mm
- net RX: track 37.0 -> 39.1 mm
- net N$6: track 24.2 -> 26.2 mm
- net SD2: track 15.0 -> 16.9 mm
- net INT: track 27.6 -> 29.2 mm
- net SCLK: track 31.8 -> 32.7 mm
- net MISO: track 30.9 -> 31.8 mm
- net GND: track 16.5 -> 15.9 mm
Other:
- board size 20.3 x 55.9 mm -> 20.3 x 58.4 mm
- board text added: "A"
- board text added: "BOOT"
- board text added: "Hail Wi-Fi"
- board text added: "RST"
